Commit message: joint fix by Emelyan

File: fanuc_custom_pkg/urdf/lrmate200id7l_macro.xacro (robot description, xacro)
@@ -191,8 +191,10 @@
       </inertial>
     </link>
-    <joint name="${prefix}tool-leftfinger" type="fixed">
-      <origin xyz="0.130 0 0.0315" rpy="0 0 0" />
+    <joint name="${prefix}tool-leftfinger" type="prismatic">
+      <origin xyz="0.130 0 0.035" rpy="0 0 0" />
       <parent link="${prefix}tool" />
       <child link="${prefix}leftfinger" />
+      <axis xyz="0 0 1"/>
+      <limit effort="100" lower="-0.0035" upper="0" velocity="0.2" />
     </joint>
     <link name="${prefix}leftfinger">
@@ -220,8 +222,10 @@
       </inertial>
     </link>
-    <joint name="${prefix}tool-rightfinger" type="fixed">
-      <origin xyz="0.130 0 -0.0315" rpy="0 0 0" />
+    <joint name="${prefix}tool-rightfinger" type="prismatic">
+      <origin xyz="0.130 0 -0.035" rpy="0 0 0" />
       <parent link="${prefix}tool" />
       <child link="${prefix}rightfinger" />
+      <axis xyz="0 0 1"/>
+      <limit effort="100" lower="0.0" upper="0.0035" velocity="0.2" />
     </joint>
     <link name="${prefix}rightfinger">
